File: PCI_ChamaMed/PCI_ChamaMed.kicad_pcb (KiCad board)
At the start: 0 parts

Commit message: Add files via upload
Parts:
- added D1: LED, LED_THT:LED_D3.0mm, F.Cu at (147.3, 111.8)
- added J1: Conn_01x02_MountingPin, Connector_BarrelJack:BarrelJack_CUI_PJ-063AH_Horizontal, F.Cu at (124.9, 119.4)
- added J2: Conn_01x01_Pin, Connector_Pin:Pin_D1.3mm_L11.0mm_LooseFit, F.Cu at (147.3, 88.9)
- added K1: RAYEX-L90S, Relay_THT:Relay_SPDT_Finder_36.11, F.Cu at (140.1, 101.6)
- added Q1: NPN, Package_TO_SOT_THT:TO-220-3_Vertical, F.Cu at (116.8, 94.0)
- added R1: R, Resistor_THT:R_Axial_DIN0207_L6.3mm_D2.5mm_P15.24mm_Horizontal, F.Cu at (124.5, 91.4)
- added R2: R, Resistor_THT:R_Axial_DIN0207_L6.3mm_D2.5mm_P15.24mm_Horizontal, F.Cu at (147.3, 109.2)
- added SW1: SW_Push, Button_Switch_THT:SW_PUSH_6mm, F.Cu at (118.8, 101.6)
- added U1: NSL-32, OptoDevice:OnSemi_CASE100AQ, F.Cu at (128.1, 86.4)
Routing:
- net Net-(Q1-E): track 0.00 -> 51.1 mm
- net Net-(D1-A): track 0.00 -> 50.7 mm
- net Net-(J1-Pin_2): track 0.00 -> 44.9 mm
- net Net-(Q1-B): track 0.00 -> 19.1 mm
- net unconnected-(J1-MountPin-PadMP): track 0.00 -> 11.2 mm
- net Net-(J2-Pin_1): track 0.00 -> 8.67 mm
- net Net-(U1-A): track 0.00 -> 6.58 mm
- net Net-(D1-K): track 0.00 -> 2.54 mm
- added copper zone on B.Cu, net Earth
Other:
- copper layers 0 -> 2
