File: PCI_ChamaMed/PCI_ChamaMed.kicad_pcb (KiCad board)
At the start: 2 copper layers, 9 parts, among them J1 Conn_01x02_MountingPin, J2 Conn_01x01_Pin, K1 RAYEX-L90S, Q1 NPN, SW1 SW_Push, U1 NSL-32

Commit message: Add files via upload
Parts:
- J1: footprint Connector_BarrelJack:BarrelJack_CUI_PJ-063AH_Horizontal -> Connector_BarrelJack:BarrelJack_CUI_PJ-102AH_Horizontal
- U1: footprint OptoDevice:OnSemi_CASE100AQ -> OptoDevice:Everlight_ITR9608-F
- moved U1 2.70 mm to (127.2, 83.8), turned to 0 degrees
- moved R1 1.91 mm to (126.4, 91.4)
- moved J1 0.72 mm to (125.6, 119.1)
Connections:
- J1 pad 1: Earth -> Net-(J1-Pin_1)
- J1 pad 2: Net-(J1-Pin_2) -> Earth
- Q1 pad 1: Net-(J1-Pin_2) -> Net-(J1-Pin_1)
- U1 pad 4: Net-(J1-Pin_2) -> Net-(J1-Pin_1)
Routing:
- net Net-(J1-Pin_1): track 0.00 -> 72.1 mm
- net Net-(J1-Pin_2): track 44.9 -> 0.00 mm
- net Net-(Q1-E): track 51.1 -> 28.0 mm
- net unconnected-(J1-MountPin-PadMP): track 11.2 -> 0.00 mm
- net Net-(Q1-B): track 19.1 -> 30.0 mm
- net Net-(U1-A): track 6.58 -> 9.00 mm
- net Net-(J2-Pin_1): track 8.67 -> 6.77 mm
- net Net-(D1-A): track 50.7 -> 51.8 mm

Commit message: Add files via upload
Parts:
- added J3: Conn_01x01_Pin, Connector_Pin:Pin_D1.3mm_L11.0mm_LooseFit, F.Cu at (148.6, 90.8)
- added J4: Conn_01x01_Pin, Connector_Pin:Pin_D1.3mm_L11.0mm_LooseFit, F.Cu at (148.6, 95.9)
- D1: value LED -> LED - 3mm
- Q1: value NPN -> MJE13007G
- R1: value R -> 220R
- R2: value R -> 680R
- moved J2 7.73 mm to (148.6, 81.3)
- moved R2 7.62 mm to (147.3, 116.8)
- moved D1 7.62 mm to (147.3, 119.4)
- moved Q1 1.31 mm to (116.5, 92.7)
- moved R1 0.63 mm to (125.7, 91.4)
Connections:
- K1 pad A1: Earth -> Net-(D1-A)
- K1 pad A2: Net-(D1-A) -> Earth
- Q1 pad 1: Net-(J1-Pin_1) -> Net-(Q1-B)
- Q1 pad 2: Net-(Q1-B) -> Net-(J1-Pin_1)
Routing:
- net Net-(D1-A): track 51.8 -> 76.8 mm
- net Net-(Q1-E): track 28.0 -> 47.4 mm
- net Net-(Q1-B): track 30.0 -> 40.9 mm
- net Net-(J2-Pin_1): track 6.77 -> 13.3 mm
- net Net-(J1-Pin_1): track 72.1 -> 71.1 mm
- net Net-(U1-A): track 9.00 -> 8.44 mm
Other:
- board text added: "Entrada"
- board text added: "GND"
- board text added: "Saída"
