File: PCI_ChamaMed/PCI_ChamaMed.kicad_sch (KiCad schematic)
At the start: 9 parts, among them J1 Conn_01x02_MountingPin, J2 Conn_01x01_Pin, K1 RAYEX-L90S, Q1 NPN, SW1 SW_Push, U1 NSL-32

Commit message: Add files via upload
Parts:
- D1: footprint (none) -> LED_THT:LED_D3.0mm
- J1: footprint (none) -> Connector_BarrelJack:BarrelJack_CUI_PJ-063AH_Horizontal
- J2: footprint (none) -> Connector_Pin:Pin_D1.3mm_L11.0mm_LooseFit
- K1: footprint Relay_THT:Relay_SPDT_RAYEX-L90S -> Relay_THT:Relay_SPDT_Finder_36.11
- R1, R2: footprint (none) -> Resistor_THT:R_Axial_DIN0207_L6.3mm_D2.5mm_P15.24mm_Horizontal
- SW1: footprint (none) -> Button_Switch_THT:SW_CW_GPTS203211B
- U1: footprint OptoDevice:Luna_NSL-32 -> OptoDevice:OnSemi_CASE100AQ
Other:
- company: (none) -> Márcio José Baldo
- title: (none) -> Placa Sinal RFID
Changed lines of the file:
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@@
 (kicad_sch (version 20230121) (generator eeschema)
   (paper "A4")
+  (title_block
+    (title "Placa Sinal RFID")
+    (date "2023-11-09")
+    (company "Márcio José Baldo")
+  )
   (junction (at 132.08 64.77) (diameter 0) (color 0 0 0 0)
   )
@@
       (effects (font (size 1.27 1.27)))
     )
-    (property "Footprint" "" (at 144.78 59.69 0)
+    (property "Footprint" "Button_Switch_THT:SW_CW_GPTS203211B" (at 144.78 59.69 0)
       (effects (font (size 1.27 1.27)) hide)
     )
@@
       (effects (font (size 1.27 1.27)) (justify right))
     )
-    (property "Footprint" "Relay_THT:Relay_SPDT_RAYEX-L90S" (at 168.91 63.5 0)
+    (property "Footprint" "Relay_THT:Relay_SPDT_Finder_36.11" (at 168.91 63.5 0)
       (effects (font (size 1.27 1.27)) (justify left) hide)
     )
@@
       (effects (font (size 1.27 1.27)) (justify right))
     )
-    (property "Footprint" "OptoDevice:Luna_NSL-32" (at 128.27 100.33 0)
+    (property "Footprint" "OptoDevice:OnSemi_CASE100AQ" (at 128.27 100.33 0)
       (effects (font (size 1.27 1.27)) hide)
     )
@@
       (effects (font (size 1.27 1.27)) (justify left))
     )
-    (property "Footprint" "" (at 116.332 116.84 90)
+    (property "Footprint" "Resistor_THT:R_Axial_DIN0207_L6.3mm_D2.5mm_P15.24mm_Horizontal" (at 116.332 116.84 90)
       (effects (font (size 1.27 1.27)) hide)
     )
@@
       (effects (font (size 1.27 1.27)) (justify right))
     )
-    (property "Footprint" "" (at 154.94 96.52 0)
+    (property "Footprint" "LED_THT:LED_D3.0mm" (at 154.94 96.52 0)
       (effects (font (size 1.27 1.27)) hide)
     )
@@
       (effects (font (size 1.27 1.27)) (justify left))
     )
-    (property "Footprint" "" (at 153.162 104.14 90)
+    (property "Footprint" "Resistor_THT:R_Axial_DIN0207_L6.3mm_D2.5mm_P15.24mm_Horizontal" (at 153.162 104.14 90)
       (effects (font (size 1.27 1.27)) hide)
     )
@@
       (effects (font (size 1.27 1.27)) (justify left))
     )
-    (property "Footprint" "" (at 96.52 91.44 0)
+    (property "Footprint" "Connector_BarrelJack:BarrelJack_CUI_PJ-063AH_Horizontal" (at 96.52 91.44 0)
       (effects (font (size 1.27 1.27)) hide)
     )
@@
       (effects (font (size 1.27 1.27)) (justify right))
     )
-    (property "Footprint" "" (at 118.11 137.16 0)
-      (effects (font (size 1.27 1.27)) hide)
-    )
+    (property "Footprint" "Connector_Pin:Pin_D1.3mm_L11.0mm_LooseFit" (at 118.11 137.16 0)
+      (effects (font (size 1.27 1.27)) hide)
+    )

Commit message: Add files via upload
Parts:
- SW1: footprint Button_Switch_THT:SW_CW_GPTS203211B -> Button_Switch_THT:SW_PUSH_6mm
Connections:
- net Earth: now reaches J1.1 (Pin_1), K1.A1, R2.2, U1.2 (K)
Changed lines of the file:
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@@
   (junction (at 175.26 44.45) (diameter 0) (color 0 0 0 0)
   )
+  (junction (at 139.7 124.46) (diameter 0) (color 0 0 0 0)
+  )
   (wire (pts (xy 154.94 124.46) (xy 154.94 107.95))
     (stroke (width 0) (type default))
@@
     (stroke (width 0) (type default))
   )
+  (wire (pts (xy 139.7 124.46) (xy 154.94 124.46))
+    (stroke (width 0) (type default))
+  )
   (wire (pts (xy 101.6 91.44) (xy 101.6 124.46))
     (stroke (width 0) (type default))
@@
     (stroke (width 0) (type default))
   )
-  (wire (pts (xy 123.19 124.46) (xy 154.94 124.46))
+  (wire (pts (xy 123.19 124.46) (xy 139.7 124.46))
     (stroke (width 0) (type default))
   )
@@
     (effects (font (size 1.27 1.27)) (justify left bottom))
   )
+  (hierarchical_label "ground" (shape input) (at 185.42 124.46 0) (fields_autoplaced)
+    (effects (font (size 1.27 1.27)) (justify left))
+  )
   (symbol (lib_id "Switch:SW_Push") (at 144.78 64.77 0) (unit 1)
     (in_bom yes) (on_board yes) (dnp no) (fields_autoplaced)
@@
       (effects (font (size 1.27 1.27)))
     )
-    (property "Footprint" "Button_Switch_THT:SW_CW_GPTS203211B" (at 144.78 59.69 0)
+    (property "Footprint" "Button_Switch_THT:SW_PUSH_6mm" (at 144.78 59.69 0)
       (effects (font (size 1.27 1.27)) hide)
     )
@@
         )
       )
+    )
+  )
+  (symbol (lib_id "power:Earth") (at 139.7 124.46 0) (unit 1)
+    (in_bom yes) (on_board yes) (dnp no) (fields_autoplaced)
+    (property "Reference" "#PWR01" (at 139.7 130.81 0)
+      (effects (font (size 1.27 1.27)) hide)
+    )
+    (property "Value" "Earth" (at 139.7 128.27 0)
+      (effects (font (size 1.27 1.27)) hide)
+    )
+    (property "Footprint" "" (at 139.7 124.46 0)
+      (effects (font (size 1.27 1.27)) hide)
+    )
+    (property "Datasheet" "~" (at 139.7 124.46 0)
+      (effects (font (size 1.27 1.27)) hide)
+    )
+    (pin "1")
+    (instances
+      (project "PCI_ChamaMed"
+        (path "/d7465849-d3ac-4f54-9d8a-6024b735dd00"
+          (reference "#PWR01") (unit 1)
+        )
+      )

Commit message: Add files via upload
Parts:
- J1: footprint Connector_BarrelJack:BarrelJack_CUI_PJ-063AH_Horizontal -> Connector_BarrelJack:BarrelJack_CUI_PJ-102AH_Horizontal
- U1: footprint OptoDevice:OnSemi_CASE100AQ -> OptoDevice:Everlight_ITR9608-F
Connections:
- net Earth: now also J1.2 (Pin_2), J1.MP (MountPin); no longer J1.1 (Pin_1)
- net at Q1.1 (C), U1.4 (R): now also J1.1 (Pin_1); no longer J1.2 (Pin_2)
Other:
- note added: "Porta digital acionada pelo Arduino. O circuito permancerá ativo se o Arduino manter o nível lógico alto (5V)"
- note removed: "Porta digital acionada pelo Arduino"
Changed lines of the file:
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@@
   (junction (at 132.08 64.77) (diameter 0) (color 0 0 0 0)
   )
+  (junction (at 154.94 64.77) (diameter 0) (color 0 0 0 0)
+  )
+  (junction (at 123.19 124.46) (diameter 0) (color 0 0 0 0)
+  )
+  (junction (at 104.14 88.9) (diameter 0) (color 0 0 0 0)
+  )
+  (junction (at 154.94 124.46) (diameter 0) (color 0 0 0 0)
+  )
+  (junction (at 175.26 44.45) (diameter 0) (color 0 0 0 0)
+  )
   (junction (at 109.22 88.9) (diameter 0) (color 0 0 0 0)
   )
-  (junction (at 154.94 64.77) (diameter 0) (color 0 0 0 0)
-  )
-  (junction (at 123.19 124.46) (diameter 0) (color 0 0 0 0)
-  )
-  (junction (at 154.94 124.46) (diameter 0) (color 0 0 0 0)
-  )
-  (junction (at 175.26 44.45) (diameter 0) (color 0 0 0 0)
-  )
   (junction (at 139.7 124.46) (diameter 0) (color 0 0 0 0)
   )
@@
     (stroke (width 0) (type default))
   )
-  (wire (pts (xy 101.6 88.9) (xy 109.22 88.9))
+  (wire (pts (xy 104.14 95.25) (xy 101.6 95.25))
     (stroke (width 0) (type default))
   )
@@
     (stroke (width 0) (type default))
   )
+  (wire (pts (xy 104.14 88.9) (xy 104.14 95.25))
+    (stroke (width 0) (type default))
+  )
   (wire (pts (xy 118.11 92.71) (xy 118.11 88.9))
     (stroke (width 0) (type default))
@@
     (stroke (width 0) (type default))
   )
-  (wire (pts (xy 101.6 91.44) (xy 101.6 124.46))
-    (stroke (width 0) (type default))
-  )
   (wire (pts (xy 109.22 64.77) (xy 114.3 64.77))
     (stroke (width 0) (type default))
@@
     (stroke (width 0) (type default))
   )
+  (wire (pts (xy 96.52 83.82) (xy 104.14 83.82))
+    (stroke (width 0) (type default))
+  )
   (wire (pts (xy 123.19 107.95) (xy 123.19 124.46))
     (stroke (width 0) (type default))
@@
     (stroke (width 0) (type default))
   )
+  (wire (pts (xy 101.6 91.44) (xy 109.22 91.44))
+    (stroke (width 0) (type default))
+  )
   (wire (pts (xy 149.86 64.77) (xy 154.94 64.77))
     (stroke (width 0) (type default))
@@
     (stroke (width 0) (type default))
   )
+  (wire (pts (xy 109.22 91.44) (xy 109.22 88.9))
+    (stroke (width 0) (type default))
+  )
+  (wire (pts (xy 101.6 88.9) (xy 104.14 88.9))
+    (stroke (width 0) (type default))
+  )
   (wire (pts (xy 172.72 80.01) (xy 132.08 80.01))
     (stroke (width 0) (type default))
@@
     (stroke (width 0) (type default))
   )
+  (wire (pts (xy 101.6 95.25) (xy 101.6 124.46))
+    (stroke (width 0) (type default))
+  )
   (wire (pts (xy 109.22 88.9) (xy 109.22 64.77))
     (stroke (width 0) (type default))
@@
     (stroke (width 0) (type default))
   )
+  (wire (pts (xy 104.14 83.82) (xy 104.14 88.9))
+    (stroke (width 0) (type default))
+  )
   (wire (pts (xy 185.42 74.93) (xy 185.42 124.46))
     (stroke (width 0) (type default))
@@
     (stroke (width 0) (type default))
   )
-  (text "Porta digital\nacionada pelo Arduino" (at 120.65 132.08 0)
+  (text "Porta digital\nacionada pelo Arduino.\nO circuito permancerá ativo\nse o Arduino manter o nível\nlógico alto (5V)"
+    (at 87.63 135.89 0)
     (effects (font (size 1.27 1.27)) (justify left bottom))
   )
@@
       (effects (font (size 1.27 1.27)) (justify right))
     )
-    (property "Footprint" "OptoDevice:OnSemi_CASE100AQ" (at 128.27 100.33 0)
+    (property "Footprint" "OptoDevice:Everlight_ITR9608-F" (at 128.27 100.33 0)
       (effects (font (size 1.27 1.27)) hide)
     )
@@
       (effects (font (size 1.27 1.27)) (justify left))
     )
-    (property "Footprint" "Connector_BarrelJack:BarrelJack_CUI_PJ-063AH_Horizontal" (at 96.52 91.44 0)
-      (effects (font (size 1.27 1.27)) hide)
-    )
+    (property "Footprint" "Connector_BarrelJack:BarrelJack_CUI_PJ-102AH_Horizontal" (at 96.52 91.44 0)
+      (effects (font (size 1.27 1.27)) hide)
+    )

Commit message: Add files via upload
Parts:
- removed Q1: NPN, Package_TO_SOT_THT:TO-220-3_Vertical, symbol Simulation_SPICE:NPN
- added J3, J4: Conn_01x01_Pin, Connector_Pin:Pin_D1.3mm_L11.0mm_LooseFit, symbol Connector:Conn_01x01_Pin
- added Q1: MJE13007G, Package_TO_SOT_THT:TO-220-3_Vertical, symbol Transistor_BJT:MJE13007G
- D1: value LED -> LED - 3mm
- R1: value R -> 220R
- R2: value R -> 680R
Connections:
- net Earth: now also K1.A2, J3.1 (Pin_1); no longer K1.A1
- net at K1.14, SW1.1: now also Q1.3 (E)
- net at D1.2 (A), K1.11, SW1.2: now also K1.A1, J4.1 (Pin_1); no longer K1.A2
- net at U1.3 (R): now also Q1.1 (B)
- net at J1.1 (Pin_1), U1.4 (R): now also Q1.2 (C)
- no-connect marks 0 -> 1
